Commit message: depth camera and ros2_controll config added
Signed-off-by: adrianCo <adrian.cobo.mh@gmail.com>

File: description/depth_camera.xacro (robot description, xacro)
@@ -26,7 +26,5 @@
     <gazebo reference="camera_link">
         <material>Gazebo/Red</material>
-        <!-- change the type to depth instead of camera if you want a RGBD camera and the image format to B8G8R8-->
-        <!-- and a min and max depth plugins params-->
-        <sensor name="camera" type="camera">
+        <sensor name="camera" type="depth">
             <pose> 0 0 0 0 0 0</pose>
             <visualize>true</visualize>
@@ -35,5 +33,5 @@
                 <horizontal_fov>1.089</horizontal_fov>
                 <image>
-                    <format>R8G8B8</format>
+                    <format>B8G8R8</format>
                     <width>640</width>
                     <height>480</height>
@@ -46,4 +44,6 @@
             <plugin name="camera_controller" filename="libgazebo_ros_camera.so">
                 <frame_name>camera_link_optical</frame_name>
+                <min_depth>0.1</min_depth>
+                <max_depth>100.0</max_depth>
             </plugin>
         </sensor>

File: description/lidar.xacro (robot description, xacro)
@@ -1,47 +1,54 @@
 <?xml version="1.0"?>
 <robot xmlns:xacro="http://www.ros.org/wiki/xacro" >
-    <joint name="camera_joint" type="fixed">
-        <origin xyz="0.305 0.0 0.08" rpy="0.0 0.0 0.0"/>
+    <joint name="laser_joint" type="fixed">
+        <origin xyz="0.1 0.0 0.175" rpy="0.0 0.0 0.0"/>
         <parent link="chassis_link"/>
-        <child link="camera_link"/>
+        <child link="laser_frame"/>
     </joint>
-    <!-- The camera is integrated on the chassis(no strick out), so there is no need of colision and inertia -->
-    <!-- It is also on a fixed joint, so there is no need of inertial component -->
-    <link name="camera_link">
+    <link name="laser_frame">
         <visual name="">
             <origin xyz="0.0 0.0 0.0" rpy="0.0 0.0 0.0"/>
             <geometry>
-                <box size="0.01 0.03 0.03"/>
+                <cylinder radius="0.05" length="0.04"/>
             </geometry>
             <material name="red" />
         </visual>
+        <collision>
+            <origin xyz="0.0 0.0 0.0" rpy="0.0 0.0 0.0"/>
+            <geometry>
+                <cylinder radius="0.05" length="0.04"/>
+            </geometry>
+        </collision>
+        <xacro:inertial_cylinder mass="0.1" length="0.04" radius="0.05">
+            <origin xyz="0.0 0.0 0.0" rpy="0.0 0.0 0.0"/>
+        </xacro:inertial_cylinder>
     </link>
-    <!-- Convert from standard roos coordinate (z to the up direction) to the camera standard coords (z point to the front)-->
-    <joint name="camera_optical_joint" type="fixed">
-        <origin xyz="0.0 0.0 0.0" rpy="${-pi/2} 0 -${pi/2}"/>
-        <parent link="camera_link"/>
-        <child link="camera_link_optical"/>
-    </joint>
-    <link name="camera_link_optical"></link>
-    <gazebo reference="camera_link">
+    <gazebo reference="laser_frame">
         <material>Gazebo/Red</material>
-        <sensor name="camera" type="camera">
+        <sensor name="laser" type="ray">
             <pose> 0 0 0 0 0 0</pose>
             <visualize>true</visualize>
             <update_rate>10</update_rate>
-            <camera>
-                <horizontal_fov>1.089</horizontal_fov>
-                <image>
-                    <format>R8G8B8</format>
-                    <width>640</width>
-                    <height>480</height>
-                </image>
-                <clip>
-                    <near>0.05</near>
-                    <far>8.0</far>
-                </clip>
-            </camera>
-            <plugin name="camera_controller" filename="libgazebo_ros_camera.so">
-                <frame_name>camera_link_optical</frame_name>
+            <ray>
+                <scan>
+                    <horizontal>
+                        <samples>360</samples>
+                        <sesolution>1</sesolution>
+                        <min_angle>-3.14</min_angle>
+                        <max_angle>3.14</max_angle>
+                    </horizontal>
+                </scan>
+                <range>
+                    <min>0.3</min>
+                    <max>12</max>
+                    <resolution>0.01</resolution>
+                </range>
+            </ray>
+            <plugin name="laser_controller" filename="libgazebo_ros_ray_sensor.so">
+                <ros>
+                    <argument>~/out:=scan</argument>
+                </ros>
+                <output_type>sensor_msgs/LaserScan</output_type>
+                <frame_name>laser_frame</frame_name>
             </plugin>
         </sensor>

File: description/robot.urdf.xacro (robot description, xacro)
@@ -2,6 +2,8 @@
 <robot xmlns:xacro="http://www.ros.org/wiki/xacro"  name="robot">
     <xacro:include filename="robot_core.xacro" />
-    <xacro:include filename="gazebo_control.xacro" />
+    <!-- <xacro:include filename="gazebo_control.xacro" /> -->
+    <xacro:include filename="ros2_control.xacro" />
     <xacro:include filename="lidar.xacro"/>
-    <xacro:include filename="camera.xacro"/>
+    <!-- <xacro:include filename="camera.xacro"/> -->
+    <xacro:include filename="depth_camera.xacro"/>
 </robot>
