Commit message: wheels controler finished
Signed-off-by: adrianCo <adrian.cobo.mh@gmail.com>

File: description/robot_core.xacro (robot description, xacro)
@@ -43,4 +43,7 @@
         </xacro:inertial_box>
     </link>
+    <gazebo reference="chassis_link">
+        <material>Gazebo/White</material>
+    </gazebo>
     <!-- LEFT WHEEL LINK -->
     <!-- continuous because it will tourn around continuously-->
@@ -71,4 +74,7 @@
         </xacro:inertial_cylinder>
     </link>
+    <gazebo reference="left_wheel_link">
+        <material>Gazebo/Blue</material>
+    </gazebo>
     <!-- RIGHT WHEEL LINK -->
     <!-- continuous because it will tourn around continuously-->
@@ -99,4 +105,7 @@
         </xacro:inertial_cylinder>
     </link>
+    <gazebo reference="right_wheel_link">
+        <material>Gazebo/Blue</material>
+    </gazebo>
     <!-- CASTER WHEEL LINK -->
     <!-- fixed because of little bit of cheating-->
@@ -125,3 +134,8 @@
         </xacro:inertial_sphere>
     </link>
+    <gazebo reference="caster_wheel_link">
+        <material>Gazebo/Black</material>
+        <mu1 value="0.0001"/>
+        <mu2 value="0.0001"/>
+    </gazebo>
 </robot>

Commit message: slam_toolbox configured
Signed-off-by: adrianCo <adrian.cobo.mh@gmail.com>

File: description/robot_core.xacro (robot description, xacro)
@@ -21,4 +21,12 @@
     <!-- Because all the geometry and turns(its going to be the center of rotation) will get easyer to get references from there-->
     <link name="base_link"></link>
+    <!-- BASE_FOOTPRINT LINK necessary for slam_toolbox-->
+    <joint name="base_footprint_joint" type="fixed">
+        <origin xyz="0.0 0.0 0.0" rpy="0.0 0.0 0.0"/>
+        <parent link="base_link"/>
+        <child link="base_footprint"/>
+    </joint>
+    <link name="base_footprint">
+    </link>
     <!-- CHASIS LINK -->
     <!-- the origin of the chassis will be just behind the center of rotation-->
