Commit message: odometri debuged
Signed-off-by: AdrianCobo <adrian.cobo.mh@gmail.com>

File: description/gazebo_control.xacro (robot description, xacro)
@@ -6,6 +6,6 @@
         <left_joint>left_wheel_joint</left_joint>
         <right_joint>right_wheel_joint</right_joint>
-        <wheel_separation>0.35</wheel_separation>
-        <wheel_diameter>0.1</wheel_diameter>
+        <wheel_separation>0.262</wheel_separation>
+        <wheel_diameter>0.7</wheel_diameter>
         <!-- Limits -->
         <max_wheel_torque>200</max_wheel_torque>

File: description/lidar.xacro (robot description, xacro)
@@ -2,5 +2,5 @@
 <robot xmlns:xacro="http://www.ros.org/wiki/xacro" >
     <joint name="laser_joint" type="fixed">
-        <origin xyz="0.165 0.0 0.185" rpy="0.0 0.0 0.0"/>
+        <origin xyz="0.165 0.0 0.185" rpy="0.0 -0.15652 0.0"/>
         <parent link="chassis_link"/>
         <child link="laser_frame"/>

File: description/real_robot_core.xacro (robot description, xacro)
@@ -64,5 +64,5 @@
     <!-- the z axis must be pointing to the horizontal and out of the robot-->
     <joint name="left_wheel_joint" type="continuous">
-        <origin xyz="0.255 0.155 0.015" rpy="-${pi/2} 0.0 0.0"/>
+        <origin xyz="0.255 0.131 0.015" rpy="-${pi/2} 0.0 0.0"/>
         <parent link="chassis_link"/>
         <child link="left_wheel_link"/>
@@ -95,5 +95,5 @@
     <!-- the z axis must be pointing to the horizontal and out of the robot-->
     <joint name="right_wheel_joint" type="continuous">
-        <origin xyz="0.255 -0.155 0.015" rpy="${pi/2} 0.0 0.0"/>
+        <origin xyz="0.255 -0.131 0.015" rpy="${pi/2} 0.0 0.0"/>
         <parent link="chassis_link"/>
         <child link="right_wheel_link"/>
