Commit message: chassis changed
Signed-off-by: AdrianCobo <adrian.cobo.mh@gmail.com>

File: description/real_robot_core.xacro (robot description, xacro)
@@ -64,6 +64,6 @@
     <!-- the z axis must be pointing to the horizontal and out of the robot-->
     <joint name="left_wheel_joint" type="continuous">
-        <origin xyz="0.0 0.155 0.0" rpy="-${pi/2} 0.0 0.0"/>
-        <parent link="base_link"/>
+        <origin xyz="0.288 0.155 0.0" rpy="-${pi/2} 0.0 0.0"/>
+        <parent link="chassis_link"/>
         <child link="left_wheel_link"/>
         <axis xyz="0.0 0.0 1.0"/>
@@ -95,6 +95,6 @@
     <!-- the z axis must be pointing to the horizontal and out of the robot-->
     <joint name="right_wheel_joint" type="continuous">
-        <origin xyz="0.0 -0.155 0.0" rpy="${pi/2} 0.0 0.0"/>
-        <parent link="base_link"/>
+        <origin xyz="0.288 -0.155 0.0" rpy="${pi/2} 0.0 0.0"/>
+        <parent link="chassis_link"/>
         <child link="right_wheel_link"/>
         <axis xyz="0.0 0.0 -1.0"/>
@@ -126,5 +126,5 @@
     <!-- the z axis must be pointing to the horizontal and out of the robot-->
     <joint name="caster_wheel_joint" type="fixed">
-        <origin xyz="0.33 0.0 -0.03" rpy="${pi/2} 0.0 0.0"/>
+        <origin xyz="0.02 0.0 -0.03" rpy="${pi/2} 0.0 0.0"/>
         <parent link="chassis_link"/>
         <child link="caster_wheel_link"/>

Commit message: xacro updated
Signed-off-by: AdrianCobo <adrian.cobo.mh@gmail.com>

File: description/real_robot_core.xacro (robot description, xacro)
@@ -126,5 +126,5 @@
     <!-- the z axis must be pointing to the horizontal and out of the robot-->
     <joint name="caster_wheel_joint" type="fixed">
-        <origin xyz="0.05 0.0 -0.00" rpy="0.0 0.0 0.0"/>
+        <origin xyz="0.05 0.0 -0.033" rpy="${pi/2} 0.0 0.0"/>
         <parent link="chassis_link"/>
         <child link="caster_wheel_link"/>
@@ -134,6 +134,5 @@
             <origin xyz="0.0 0.0 0.0" rpy="0.0 0.0 0.0"/>
             <geometry>
-                <!-- <cylinder radius="0.02" length="0.018"/> -->
-                <mesh filename="/home/acobo/Desktop/ros2_ws/src/my_bot/meshes/caster_wheel/caster_wheel.dae" uri="model://home/acobo/Desktop/ros2_ws/src/my_bot/meshes/caster_wheel/testing_freecad_color.dae" scale="0.001 0.001 0.001"/>
+                <cylinder radius="0.0175" length="0.018"/>
             </geometry>
         </visual>
@@ -141,8 +140,8 @@
             <origin xyz="0.0 0.0 0.0" rpy="0.0 0.0 0.0"/>
             <geometry>
-                <mesh filename="/home/acobo/Desktop/ros2_ws/src/my_bot/meshes/caster_wheel/caster_wheel.stl" scale="0.001 0.001 0.001"/>
+                <cylinder radius="0.0175" length="0.018"/>
             </geometry>
         </collision>
-        <xacro:inertial_cylinder mass="0.1" length="0.018" radius="0.035">
+        <xacro:inertial_cylinder mass="0.1" length="0.018" radius="0.0175">
             <origin xyz="0.0 0.0 0.0" rpy="0.0 0.0 0.0"/>
         </xacro:inertial_cylinder>

Commit message: lidar model and caster wheel model added. Needs to solve problem with color and rviz
Signed-off-by: AdrianCobo <adrian.cobo.mh@gmail.com>

File: description/real_robot_core.xacro (robot description, xacro)
@@ -126,5 +126,5 @@
     <!-- the z axis must be pointing to the horizontal and out of the robot-->
     <joint name="caster_wheel_joint" type="fixed">
-        <origin xyz="0.05 0.0 -0.033" rpy="${pi/2} 0.0 0.0"/>
+        <origin xyz="0.05 0.0 0.0" rpy="0.0 0.0 0.0"/>
         <parent link="chassis_link"/>
         <child link="caster_wheel_link"/>
@@ -134,5 +134,6 @@
             <origin xyz="0.0 0.0 0.0" rpy="0.0 0.0 0.0"/>
             <geometry>
-                <cylinder radius="0.0175" length="0.018"/>
+                <!-- <cylinder radius="0.0175" length="0.018"/> -->
+                <mesh filename="/home/acobo/Desktop/ros2_ws/src/my_bot/meshes/caster_wheel/caster_wheel.dae" scale="0.001 0.001 0.001"/>
             </geometry>
         </visual>
@@ -140,5 +141,5 @@
             <origin xyz="0.0 0.0 0.0" rpy="0.0 0.0 0.0"/>
             <geometry>
-                <cylinder radius="0.0175" length="0.018"/>
+                <mesh filename="/home/acobo/Desktop/ros2_ws/src/my_bot/meshes/caster_wheel/caster_wheel.stl" scale="0.001 0.001 0.001"/>
             </geometry>
         </collision>

Commit message: chassis link corrected
Signed-off-by: AdrianCobo <adrian.cobo.mh@gmail.com>

File: description/real_robot_core.xacro (robot description, xacro)
@@ -23,4 +23,5 @@
     <!-- Using diferential mobile robots its better to use de center of the two wheels as the base link-->
     <!-- Because all the geometry and turns(its going to be the center of rotation) will get easyer to get references from there-->
+    <!-- The base_link is usually the chassis or body of a robot that is immediately attached to the ground or world reference frame. -->
     <link name="base_link"></link>
     <!-- BASE_FOOTPRINT LINK necessary for slam_toolbox-->
@@ -34,6 +35,8 @@
     <!-- CHASIS LINK -->
     <!-- the origin of the chassis will be just behind the center of rotation-->
+    <!-- as the caster wheel is higher, the box is rotated in y -->
+    <!-- the mass is created based on the joint, not the link -->
     <joint name="chase_joint" type="fixed">
-        <origin xyz="-0.255 0.0 0.0" rpy="0.0 0.0 0.0"/>
+        <origin xyz="-0.255 0.0 0.06" rpy="0.0 0.15652 0.0"/>
         <parent link="base_link"/>
         <child link="chassis_link"/>
@@ -48,11 +51,11 @@
         </visual>
         <collision>
-            <origin xyz="0.165 0.0 0.06" rpy="0.0 0.0 0.0"/>
+            <origin xyz="0.16 0.0 0.07" rpy="0.0 0.0 0.0"/>
             <geometry>
                 <box size="0.32 0.225 0.14"/>
             </geometry>
         </collision>
-        <xacro:inertial_box mass="0.5" x="0.33" y="0.225" z="0.12">
-            <origin xyz="0.165 0.0 0.06" rpy="0.0 0.0 0.0"/>
+        <xacro:inertial_box mass="0.5" x="0.32" y="0.225" z="0.14">
+            <origin xyz="0.165 0.0 0.0" rpy="0.0 0.0 0.0"/>
         </xacro:inertial_box>
     </link>

Commit message: gazebo and rviz mesh problem solved
Signed-off-by: AdrianCobo <adrian.cobo.mh@gmail.com>

File: description/real_robot_core.xacro (robot description, xacro)
@@ -135,11 +135,12 @@
             <geometry>
                 <!-- <cylinder radius="0.0175" length="0.018"/> -->
-                <mesh filename="/home/acobo/Desktop/ros2_ws/src/my_bot/meshes/caster_wheel/caster_wheel.dae" scale="0.001 0.001 0.001"/>
+                <mesh filename="package://my_bot/meshes/caster_wheel/caster_wheel.stl" scale="0.001 0.001 0.001"/>
             </geometry>
+            <material name="blue" />
         </visual>
         <collision>
             <origin xyz="0.0 0.0 0.0" rpy="0.0 0.0 0.0"/>
             <geometry>
-                <mesh filename="/home/acobo/Desktop/ros2_ws/src/my_bot/meshes/caster_wheel/caster_wheel.stl" scale="0.001 0.001 0.001"/>
+                <mesh filename="package://my_bot/meshes/caster_wheel/caster_wheel.stl" scale="0.001 0.001 0.001"/>
             </geometry>
         </collision>
@@ -149,4 +150,5 @@
     </link>
     <gazebo reference="caster_wheel_link">
+        <material>Gazebo/Blue</material>
         <mu1 value="0.0001"/>
         <mu2 value="0.0001"/>

Commit message: .dae is better
Signed-off-by: AdrianCobo <adrian.cobo.mh@gmail.com>

File: description/real_robot_core.xacro (robot description, xacro)
@@ -135,12 +135,11 @@
             <geometry>
                 <!-- <cylinder radius="0.0175" length="0.018"/> -->
-                <mesh filename="package://my_bot/meshes/caster_wheel/caster_wheel.stl" scale="0.001 0.001 0.001"/>
+                <mesh filename="package://my_bot/meshes/caster_wheel/caster_wheel.dae" scale="0.001 0.001 0.001"/>
             </geometry>
-            <material name="blue" />
         </visual>
         <collision>
             <origin xyz="0.0 0.0 0.0" rpy="0.0 0.0 0.0"/>
             <geometry>
-                <mesh filename="package://my_bot/meshes/caster_wheel/caster_wheel.stl" scale="0.001 0.001 0.001"/>
+                <mesh filename="package://my_bot/meshes/caster_wheel/caster_wheel.dae" scale="0.001 0.001 0.001"/>
             </geometry>
         </collision>
@@ -150,5 +149,4 @@
     </link>
     <gazebo reference="caster_wheel_link">
-        <material>Gazebo/Blue</material>
         <mu1 value="0.0001"/>
         <mu2 value="0.0001"/>

Commit message: caster wheel color
Signed-off-by: AdrianCobo <adrian.cobo.mh@gmail.com>

File: description/real_robot_core.xacro (robot description, xacro)
@@ -141,5 +141,5 @@
             <origin xyz="0.0 0.0 0.0" rpy="0.0 0.0 0.0"/>
             <geometry>
-                <mesh filename="package://my_bot/meshes/caster_wheel/caster_wheel.dae" scale="0.001 0.001 0.001"/>
+                <mesh filename="package://my_bot/meshes/caster_wheel/caster_wheel.stl" scale="0.001 0.001 0.001"/>
             </geometry>
         </collision>
