Commit message: laser y camera xacro changed
Signed-off-by: AdrianCobo <adrian.cobo.mh@gmail.com>

File: description/camera.xacro (robot description, xacro)
@@ -2,5 +2,5 @@
 <robot xmlns:xacro="http://www.ros.org/wiki/xacro" >
     <joint name="camera_joint" type="fixed">
-        <origin xyz="0.305 0.0 0.08" rpy="0.0 0.0 0.0"/>
+        <origin xyz="0.33 -0.0255 0.08" rpy="0.0 0.0 0.0"/>
         <parent link="chassis_link"/>
         <child link="camera_link"/>

File: description/lidar.xacro (robot description, xacro)
@@ -2,5 +2,5 @@
 <robot xmlns:xacro="http://www.ros.org/wiki/xacro" >
     <joint name="laser_joint" type="fixed">
-        <origin xyz="0.1 0.0 0.175" rpy="0.0 0.0 0.0"/>
+        <origin xyz="0.16 0.0 0.175" rpy="0.0 0.0 0.0"/>
         <parent link="chassis_link"/>
         <child link="laser_frame"/>

File: description/real_robot.urdf.xacro (robot description, xacro)
@@ -11,5 +11,5 @@
     </xacro:unless>
     <xacro:include filename="lidar.xacro"/>
-    <!-- <xacro:include filename="camera.xacro"/> -->
-    <xacro:include filename="depth_camera.xacro"/>
+    <!-- <xacro:include filename="depth_camera.xacro"/> -->
+    <xacro:include filename="camera.xacro"/>
 </robot>

Commit message: caster_wheel added
Signed-off-by: AdrianCobo <adrian.cobo.mh@gmail.com>

File: description/camera.xacro (robot description, xacro)
@@ -2,5 +2,5 @@
 <robot xmlns:xacro="http://www.ros.org/wiki/xacro" >
     <joint name="camera_joint" type="fixed">
-        <origin xyz="0.33 -0.0255 0.08" rpy="0.0 0.0 0.0"/>
+        <origin xyz="0.32 -0.06 0.095" rpy="0.0 0.0 0.0"/>
         <parent link="chassis_link"/>
         <child link="camera_link"/>

File: description/lidar.xacro (robot description, xacro)
@@ -2,5 +2,5 @@
 <robot xmlns:xacro="http://www.ros.org/wiki/xacro" >
     <joint name="laser_joint" type="fixed">
-        <origin xyz="0.16 0.0 0.175" rpy="0.0 0.0 0.0"/>
+        <origin xyz="0.165 0.0 0.185" rpy="0.0 0.0 0.0"/>
         <parent link="chassis_link"/>
         <child link="laser_frame"/>

File: description/real_robot_core.xacro (robot description, xacro)
@@ -35,5 +35,5 @@
     <!-- the origin of the chassis will be just behind the center of rotation-->
     <joint name="chase_joint" type="fixed">
-        <origin xyz="-0.1 0.0 0.0" rpy="0.0 0.0 0.0"/>
+        <origin xyz="-0.255 0.0 0.0" rpy="0.0 0.0 0.0"/>
         <parent link="base_link"/>
         <child link="chassis_link"/>
@@ -41,7 +41,7 @@
     <link name="chassis_link">
         <visual name="">
-            <origin xyz="0.165 0.0 0.06" rpy="0.0 0.0 0.0"/>
+            <origin xyz="0.16 0.0 0.07" rpy="0.0 0.0 0.0"/>
             <geometry>
-                <box size="0.33 0.225 0.12"/>
+                <box size="0.32 0.225 0.14"/>
             </geometry>
             <material name="grey"/>
@@ -50,5 +50,5 @@
             <origin xyz="0.165 0.0 0.06" rpy="0.0 0.0 0.0"/>
             <geometry>
-                <box size="0.33 0.225 0.12"/>
+                <box size="0.32 0.225 0.14"/>
             </geometry>
         </collision>
@@ -64,5 +64,5 @@
     <!-- the z axis must be pointing to the horizontal and out of the robot-->
     <joint name="left_wheel_joint" type="continuous">
-        <origin xyz="0.288 0.155 0.0" rpy="-${pi/2} 0.0 0.0"/>
+        <origin xyz="0.255 0.155 0.015" rpy="-${pi/2} 0.0 0.0"/>
         <parent link="chassis_link"/>
         <child link="left_wheel_link"/>
@@ -74,5 +74,5 @@
             <origin xyz="0.0 0.0 0.0" rpy="0.0 0.0 0.0"/>
             <geometry>
-                <cylinder radius="0.035" length="0.029"/>
+                <cylinder radius="0.035" length="0.027"/>
             </geometry>
             <material name="blue" />
@@ -81,8 +81,8 @@
             <origin xyz="0.0 0.0 0.0" rpy="0.0 0.0 0.0"/>
             <geometry>
-                <cylinder radius="0.035" length="0.029"/>
+                <cylinder radius="0.035" length="0.027"/>
             </geometry>
         </collision>
-        <xacro:inertial_cylinder mass="0.1" length="0.029" radius="0.035">
+        <xacro:inertial_cylinder mass="0.1" length="0.027" radius="0.035">
             <origin xyz="0.0 0.0 0.0" rpy="0.0 0.0 0.0"/>
         </xacro:inertial_cylinder>
@@ -95,5 +95,5 @@
     <!-- the z axis must be pointing to the horizontal and out of the robot-->
     <joint name="right_wheel_joint" type="continuous">
-        <origin xyz="0.288 -0.155 0.0" rpy="${pi/2} 0.0 0.0"/>
+        <origin xyz="0.255 -0.155 0.015" rpy="${pi/2} 0.0 0.0"/>
         <parent link="chassis_link"/>
         <child link="right_wheel_link"/>
@@ -105,5 +105,5 @@
             <origin xyz="0.0 0.0 0.0" rpy="0.0 0.0 0.0"/>
             <geometry>
-                <cylinder radius="0.035" length="0.029"/>
+                <cylinder radius="0.035" length="0.027"/>
             </geometry>
             <material name="blue" />
@@ -112,8 +112,8 @@
             <origin xyz="0.0 0.0 0.0" rpy="0.0 0.0 0.0"/>
             <geometry>
-                <cylinder radius="0.035" length="0.029"/>
+                <cylinder radius="0.035" length="0.027"/>
             </geometry>
         </collision>
-        <xacro:inertial_cylinder mass="0.1" length="0.035" radius="0.029">
+        <xacro:inertial_cylinder mass="0.1" length="0.027" radius="0.035">
             <origin xyz="0.0 0.0 0.0" rpy="0.0 0.0 0.0"/>
         </xacro:inertial_cylinder>
@@ -126,5 +126,5 @@
     <!-- the z axis must be pointing to the horizontal and out of the robot-->
     <joint name="caster_wheel_joint" type="fixed">
-        <origin xyz="0.02 0.0 -0.03" rpy="${pi/2} 0.0 0.0"/>
+        <origin xyz="0.05 0.0 -0.00" rpy="0.0 0.0 0.0"/>
         <parent link="chassis_link"/>
         <child link="caster_wheel_link"/>
@@ -134,20 +134,19 @@
             <origin xyz="0.0 0.0 0.0" rpy="0.0 0.0 0.0"/>
             <geometry>
-                <cylinder radius="0.02" length="0.018"/>
+                <!-- <cylinder radius="0.02" length="0.018"/> -->
+                <mesh filename="/home/acobo/Desktop/ros2_ws/src/my_bot/meshes/caster_wheel/caster_wheel.dae" uri="model://home/acobo/Desktop/ros2_ws/src/my_bot/meshes/caster_wheel/testing_freecad_color.dae" scale="0.001 0.001 0.001"/>
             </geometry>
-            <material name="black" />
         </visual>
         <collision>
             <origin xyz="0.0 0.0 0.0" rpy="0.0 0.0 0.0"/>
             <geometry>
-                <cylinder radius="0.02" length="0.018"/>
+                <mesh filename="/home/acobo/Desktop/ros2_ws/src/my_bot/meshes/caster_wheel/caster_wheel.stl" scale="0.001 0.001 0.001"/>
             </geometry>
         </collision>
-        <xacro:inertial_cylinder mass="0.1" length="0.018" radius="0.02">
+        <xacro:inertial_cylinder mass="0.1" length="0.018" radius="0.035">
             <origin xyz="0.0 0.0 0.0" rpy="0.0 0.0 0.0"/>
         </xacro:inertial_cylinder>
     </link>
     <gazebo reference="caster_wheel_link">
-        <material>Gazebo/Black</material>
         <mu1 value="0.0001"/>
         <mu2 value="0.0001"/>

Commit message: jazzy update
Signed-off-by: adrianCo <adrian.cobo.mh@gmail.com>

File: description/camera.xacro (robot description, xacro)
@@ -33,4 +33,5 @@
             <update_rate>10</update_rate>
             <camera>
+                <camera_info_topic>camera/camera_info</camera_info_topic>
                 <horizontal_fov>1.089</horizontal_fov>
                 <image>
@@ -44,7 +45,6 @@
                 </clip>
             </camera>
-            <plugin name="camera_controller" filename="libgazebo_ros_camera.so">
-                <frame_name>camera_link_optical</frame_name>
-            </plugin>
+            <topic>camera/image_raw</topic>
+            <gz_frame_id>camera_link_optical</gz_frame_id>
         </sensor>
     </gazebo>

File: description/gazebo_control.xacro (robot description, xacro)
@@ -2,19 +2,27 @@
 <robot xmlns:xacro="http://www.ros.org/wiki/xacro" >
 <gazebo>
-    <plugin name="diff_drive" filename="libgazebo_ros_diff_drive.so">
+    <plugin name="gz::sim::systems::DiffDrive" filename="gz-sim-diff-drive-system">
         <!-- Wheel information -->
         <left_joint>left_wheel_joint</left_joint>
         <right_joint>right_wheel_joint</right_joint>
         <wheel_separation>0.262</wheel_separation>
-        <wheel_diameter>0.7</wheel_diameter>
+        <wheel_radius>0.35</wheel_radius>
         <!-- Limits -->
-        <max_wheel_torque>200</max_wheel_torque>
-        <max_wheel_acceleration>10.0</max_wheel_acceleration>
+        <!-- <max_wheel_torque>200</max_wheel_torque> -->
+        <max_linear_acceleration>10.0</max_linear_acceleration>
+        <!--input-->
+        <topic>cmd_vel</topic>
         <!-- Output -->
-        <odometry_frame>odom</odometry_frame>
-        <robot_base_frame>base_link</robot_base_frame>
-        <publish_odom>true</publish_odom>
-        <publish_odom_tf>true</publish_odom_tf>
-        <publish_wheel_tf>true</publish_wheel_tf>
+        <frame_id>odom</frame_id>
+        <child_frame_id>base_link</child_frame_id>
+        <odom_topic>odom</odom_topic>
+        <odom_publisher_frequency>30</odom_publisher_frequency>
+        <tf_topic>/tf</tf_topic>
+    </plugin>
+    <plugin filename="gz-sim-joint-state-publisher-system"
+        name="gz::sim::systems::JointStatePublisher">
+        <topic>joint_states</topic>
+        <joint_name>left_wheel_joint</joint_name>
+        <joint_name>right_wheel_joint</joint_name>
     </plugin>
 </gazebo>

File: description/lidar.xacro (robot description, xacro)
@@ -26,9 +26,9 @@
     <gazebo reference="laser_frame">
         <material>Gazebo/Red</material>
-        <sensor name="laser" type="ray">
+        <sensor name="laser" type="gpu_lidar">
             <pose> 0 0 0 0 0 0</pose>
             <visualize>false</visualize>
             <update_rate>10</update_rate>
-            <ray>
+            <lidar>
                 <scan>
                     <horizontal>
@@ -43,12 +43,7 @@
                     <resolution>0.01</resolution>
                 </range>
-            </ray>
-            <plugin name="laser_controller" filename="libgazebo_ros_ray_sensor.so">
-                <ros>
-                    <argument>~/out:=scan</argument>
-                </ros>
-                <output_type>sensor_msgs/LaserScan</output_type>
-                <frame_name>laser_frame</frame_name>
-            </plugin>
+            </lidar>
+            <topic>scan</topic>
+            <gz_frame_id>laser_frame</gz_frame_id>
         </sensor>
     </gazebo>

File: description/real_robot_core.xacro (robot description, xacro)
@@ -71,5 +71,4 @@
         <child link="left_wheel_link"/>
         <axis xyz="0.0 0.0 1.0"/>
-        <limit lower="0.0" upper="0.0" effort="0.0" velocity="0.0"/>
     </joint>
     <link name="left_wheel_link">
@@ -102,5 +101,4 @@
         <child link="right_wheel_link"/>
         <axis xyz="0.0 0.0 -1.0"/>
-        <limit lower="0.0" upper="0.0" effort="0.0" velocity="0.0"/>
     </joint>
     <link name="right_wheel_link">
@@ -138,5 +136,5 @@
             <geometry>
                 <!-- <cylinder radius="0.0175" length="0.018"/> -->
-                <mesh filename="package://my_bot/meshes/caster_wheel/caster_wheel.dae" scale="0.001 0.001 0.001"/>
+                <mesh filename="model://my_bot/meshes/caster_wheel/caster_wheel.dae" scale="0.001 0.001 0.001"/>
             </geometry>
         </visual>
@@ -144,5 +142,5 @@
             <origin xyz="0.0 0.0 0.0" rpy="0.0 0.0 0.0"/>
             <geometry>
-                <mesh filename="package://my_bot/meshes/caster_wheel/caster_wheel.stl" scale="0.001 0.001 0.001"/>
+                <mesh filename="model://my_bot/meshes/caster_wheel/caster_wheel.stl" scale="0.001 0.001 0.001"/>
             </geometry>
         </collision>

File: description/robot.urdf.xacro (robot description, xacro)
@@ -1,7 +1,13 @@
 <?xml version="1.0"?>
 <robot xmlns:xacro="http://www.ros.org/wiki/xacro"  name="robot">
+    <xacro:arg name="use_ros2_control" default="true"/>
+    <xacro:arg name="sim_mode" default="false"/>
     <xacro:include filename="robot_core.xacro" />
-    <!-- <xacro:include filename="gazebo_control.xacro" /> -->
-    <xacro:include filename="ros2_control.xacro" />
+     <xacro:if value="$(arg use_ros2_control)">
+        <xacro:include filename="ros2_control.xacro" />
+    </xacro:if>
+    <xacro:unless value="$(arg use_ros2_control)">
+        <xacro:include filename="gazebo_control.xacro" />
+    </xacro:unless>
     <xacro:include filename="lidar.xacro"/>
     <!-- <xacro:include filename="camera.xacro"/> -->

File: description/ros2_control.xacro (robot description, xacro)
@@ -16,4 +16,6 @@
             <joint name="left_wheel_joint">
                 <command_interface name="velocity"/>
+                    <param name="min">-10</param>
+                    <param name="max">10</param>
                 <state_interface name="position"/>
                 <state_interface name="velocity"/>
@@ -21,4 +23,6 @@
             <joint name="right_wheel_joint">
                 <command_interface name="velocity"/>
+                    <param name="min">-10</param>
+                    <param name="max">10</param>
                 <state_interface name="position"/>
                 <state_interface name="velocity"/>
@@ -29,5 +33,5 @@
         <ros2_control name="GazeboSystem" type="system">
             <hardware>
-                <plugin>gazebo_ros2_control/GazeboSystem</plugin>
+                <plugin>gz_ros2_control/GazeboSimSystem</plugin>
             </hardware>
             <joint name="left_wheel_joint">
@@ -50,5 +54,5 @@
     </xacro:if>
     <gazebo>
-        <plugin name="gazebo_ros2_control" filename="libgazebo_ros2_control.so">
+        <plugin name="gz_ros2_control::GazeboSimROS2ControlPlugin" filename="libgz_ros2_control-system.so">
             <parameters>$(find my_bot)/config/my_controllers.yaml</parameters>
             <parameters>$(find my_bot)/config/gaz_ros2_ctl_use_sim.yaml</parameters>
